Commit message: 0914

File: mobile_manipulator/urdf/base.xacro (robot description, xacro)
@@ -2,290 +2,289 @@
 <robot name="tracer_mini" xmlns:xacro="http://www.ros.org/wiki/xacro">
   <xacro:property name="connection_link" value="base_arm_connector" />
-  <xacro:property name="M_PI" value="3.14159265358979323846" />
-  <xacro:property name="base_body_width" value="0.4" />
-  <xacro:property name="base_body_length" value="0.4" />
-  <xacro:property name="total_height" value="0.29386" />
-  <!-- <xacro:property name="base_body_height" value="0.26344" /> -->
-  <!-- <xacro:property name="floor_to_base_height" value="0.03042" /> -->
-  <xacro:property name="front_wheel_length" value="0.127547" />
-  <xacro:property name="front_wheel_radius" value="0.0575" />
-  <xacro:property name="front_wheel_depth" value="0.079536242431022" />
-  <xacro:property name="rear_wheel_length" value="0.125" />
-  <xacro:property name="rear_wheel_radius" value="0.0325" />
-  <xacro:property name="rear_wheel_depth" value="0.022335230282742743" />
-  <!-- About the mass ratio of each part: -->
-  <!-- <xacro:property name="total_mass" value="27.5289014037350" /> -->
-  <xacro:property name="base_body_mass" value="24.3948952632956" />
-  <xacro:property name="front_wheel_mass" value="1.0568406891164" />
-  <xacro:property name="rear_wheel_bracket_mass" value="0.0211573699864" />
-  <xacro:property name="rear_wheel_mass" value="0.0920111896829" />
-  <xacro:property name="camera_mass" value="0.2333248928640" />
-  <xacro:property name="lidar_mass" value="0.1071556446529" />
-  <xacro:property name="base_arm_connector_mass" value="0.4535071053510" />
-  <!-- Include inertial xacro files -->
-  <xacro:include filename="$(find mobile_manipulator)/urdf/inertial.xacro" />
-  <link name="base_link"/>
-  <joint name="base_body_joint" type="fixed">
-    <origin xyz="0 0 ${total_height}" rpy="0 0 0" />
-    <parent link="base_link" />
-    <child link="base_body" />
-    <axis xyz="0 0 0" />
-  </joint>
-  <link name="base_body">
-    <visual>
-      <origin xyz="0 0 0" rpy="0 0 0" />
-      <geometry>
-        <mesh filename="package://mobile_manipulator/meshes/base/base_body.stl" />
-      </geometry>
-      <material name="">
-        <color rgba="1 1 1 1" />
-      </material>
-    </visual>
-    <collision>
-       <origin xyz="0 0 0" rpy="0 0 0" />
-      <geometry>
-        <mesh filename="package://mobile_manipulator/meshes/base/base_body.stl" />
-      </geometry>
-    </collision>
-    <xacro:inertial_box mass="${base_body_mass}" x="0.4" y="0.4" z="0.26344">
-      <origin xyz="0 0 0" rpy="0 0 0" />
-    </xacro:inertial_box>
-  </link>
-  <joint name="fl_joint" type="continuous">
-    <origin xyz="0.05 ${front_wheel_length} ${front_wheel_radius - total_height} " rpy="-${M_PI / 2} 0 0"/>
-    <parent link="base_body" />
-    <child link="fl_wheel" />
-    <axis xyz="0 0 1" />
-  </joint>
-  <link name="fl_wheel">
-    <visual>
-      <origin rpy="${M_PI/2} 0 0" xyz="0 0 0" />
-      <geometry>
-        <mesh filename="package://mobile_manipulator/meshes/base/front_wheel.stl" />
-      </geometry>
-      <material name="">
-        <color rgba="0.5 0.5 0.5 1" />
-      </material>
-    </visual>
-    <collision>
-      <origin rpy="${M_PI/2} 0 0" xyz="0 0 0" />
-      <geometry>
-        <mesh filename="package://mobile_manipulator/meshes/base/front_wheel.stl" />
-      </geometry>
-    </collision>
-    <xacro:inertial_cylinder mass="${front_wheel_mass}" length="${front_wheel_depth}" radius="${front_wheel_radius}">
-      <origin rpy="${M_PI/2} 0 0" xyz="0 0 0" />
-    </xacro:inertial_cylinder>
-  </link>
-  <joint name="fr_joint" type="continuous">
-    <origin xyz="0.05 -${front_wheel_length} ${front_wheel_radius - total_height}" rpy="${M_PI/2} 0 0" />
-    <parent link="base_body" />
-    <child link="fr_wheel" />
-    <axis xyz="0 0 1" />
-  </joint>
-  <link name="fr_wheel">
-    <visual>
-      <origin rpy="-${M_PI/2} 0 0" xyz="0 0 0" />
-      <geometry>
-        <mesh filename="package://mobile_manipulator/meshes/base/front_wheel.stl" />
-      </geometry>
-      <material name="">
-        <color rgba="0.5 0.5 0.5 1" />
-      </material>
-    </visual>
-    <collision>
-      <origin rpy="-${M_PI/2} 0 0" xyz="0 0 0" />
-      <geometry>
-        <mesh filename="package://mobile_manipulator/meshes/base/front_wheel.stl" />
-      </geometry>
-    </collision>
-    <xacro:inertial_cylinder mass="${front_wheel_mass}" length="${front_wheel_depth}" radius="${front_wheel_radius}">
-      <origin rpy="-${M_PI/2} 0 0" xyz="0 0 0" />
-    </xacro:inertial_cylinder>
-  </link>
-  <joint name="rl_bracket_joint" type="continuous">
-    <origin xyz="-0.17043 ${rear_wheel_length} ${rear_wheel_radius - total_height + 0.0453}" rpy="0 0 0" />
-    <parent link="base_body" />
-    <child link="rl_bracket" />
-    <axis xyz="0 0 1" />
-  </joint>
-  <link name="rl_bracket">
-    <visual>
-      <origin rpy="0 0 ${M_PI/2}" xyz="0 0 0" />
-      <geometry>
-        <mesh filename="package://mobile_manipulator/meshes/base/rear_wheel_bracket.stl" />
-      </geometry>
-      <material name="">
-        <color rgba="0.5 0.5 0.5 1" />
-      </material>
-    </visual>
-    <collision>
-      <origin rpy="0 0 ${M_PI/2}" xyz="0 0 0" />
-      <geometry>
-        <mesh filename="package://mobile_manipulator/meshes/base/rear_wheel_bracket.stl" />
-      </geometry>
-    </collision>
-    <xacro:inertial_cylinder mass="${rear_wheel_bracket_mass}" length="0.0453" radius="0.01">
-      <origin rpy="0 0 ${M_PI/2}" xyz="0 0 0" />
-    </xacro:inertial_cylinder>
-  </link>
-  <joint name="rl_wheel_joint" type="continuous">
-    <origin xyz="-0.027 0 -0.0453" rpy="-${M_PI/2} 0 0" />
-    <parent link="rl_bracket" />
-    <child link="rl_wheel" />
-    <axis xyz="0 0 1" />
-  </joint>
-  <link name="rl_wheel">
-    <visual>
-      <origin rpy="0 -${M_PI/2} 0" xyz="0 0 0" />
-      <geometry>
-        <mesh filename="package://mobile_manipulator/meshes/base/rear_wheel.stl" />
-      </geometry>
-      <material name="">
-        <color rgba="0.5 0.5 0.5 1" />
-      </material>
-    </visual>
-    <collision>
-      <origin rpy="0 -${M_PI/2} 0" xyz="0 0 0" />
-      <geometry>
-        <mesh filename="package://mobile_manipulator/meshes/base/rear_wheel.stl" />
-      </geometry>
-    </collision>
-    <xacro:inertial_cylinder mass="${rear_wheel_mass}" length="${rear_wheel_depth}" radius="${rear_wheel_radius}">
-      <origin rpy="0 -${M_PI/2} 0" xyz="0 0 0" />
-    </xacro:inertial_cylinder>
-  </link>
-  <joint name="rr_bracekt_joint" type="continuous">
-    <origin xyz="-0.17043 -${rear_wheel_length} ${rear_wheel_radius - total_height + 0.0453}" rpy="0 0 0" />
-    <parent link="base_body" />
-    <child link="rr_bracket" />
-    <axis xyz="0 0 1" />
-  </joint>
-  <link name="rr_bracket">
-    <visual>
-      <origin rpy="0 0 ${M_PI/2}" xyz="0 0 0" />
-      <geometry>
-        <mesh filename="package://mobile_manipulator/meshes/base/rear_wheel_bracket.stl" />
-      </geometry>
-      <material name="">
-        <color rgba="0.5 0.5 0.5 1" />
-      </material>
-    </visual>
-    <collision>
-      <origin rpy="0 0 ${M_PI/2}" xyz="0 0 0" />
-      <geometry>
-        <mesh filename="package://mobile_manipulator/meshes/base/rear_wheel_bracket.stl" />
-      </geometry>
-    </collision>
-    <xacro:inertial_cylinder mass="${rear_wheel_bracket_mass}" length="0.0453" radius="0.01">
-      <origin rpy="0 0 ${M_PI/2}" xyz="0 0 0" />
-    </xacro:inertial_cylinder>
-  </link>
-  <joint name="rr_wheel_joint" type="continuous">
-    <origin xyz="-0.027 0 -0.0453" rpy="${M_PI/2} 0 0" />
-    <parent link="rr_bracket" />
-    <child link="rr_wheel" />
-    <axis xyz="0 0 1" />
-  </joint>
-  <link name="rr_wheel">
-    <visual>
-      <origin rpy="0 ${M_PI/2} 0" xyz="0 0 0" />
-      <geometry>
-        <mesh filename="package://mobile_manipulator/meshes/base/rear_wheel.stl" />
-      </geometry>
-      <material name="">
-        <color rgba="0.5 0.5 0.5 1" />
-      </material>
-    </visual>
-    <collision>
-      <origin rpy="0 ${M_PI/2} 0" xyz="0 0 0" />
-      <geometry>
-        <mesh filename="package://mobile_manipulator/meshes/base/rear_wheel.stl" />
-      </geometry>
-    </collision>
-    <xacro:inertial_cylinder mass="${rear_wheel_mass}" length="${rear_wheel_depth}" radius="${rear_wheel_radius}">
-      <origin rpy="0 ${M_PI/2} 0" xyz="0 0 0" />
-    </xacro:inertial_cylinder>
-  </link>
-  <joint name="laser_joint" type="fixed">
-    <origin xyz="0.04517 0 -0.1053" rpy="0 0 0" />
-    <parent link="base_body" />
-    <child link="laser_Link" />
-    <axis xyz="0 0 0" />
-  </joint>
-  <link name="laser_Link">
-    <visual>
-      <origin xyz="0 0 0" rpy="0 0 0" />
-      <geometry>
-        <mesh filename="package://mobile_manipulator/meshes/base/lidar.stl" />
-      </geometry>
-      <material name="">
-        <color rgba="1 0.6 0 1" />
-      </material>
-    </visual>
-    <collision>
-      <origin xyz="0 0 0" rpy="0 0 0" />
-      <geometry>
-        <mesh filename="package://mobile_manipulator/meshes/base/lidar.stl" />
-      </geometry>
-    </collision>
-    <xacro:inertial_cylinder mass="${lidar_mass}" length="0.02" radius="0.0389">
-      <origin xyz="0 0 0" rpy="0 0 0" />
-    </xacro:inertial_cylinder>
-  </link>
-  <joint name="camera_joint" type="fixed">
-    <origin xyz="0.115 0 -0.04565" rpy="0 0 0" />
-    <parent link="base_body" />
-    <child link="camera_link" />
-    <axis xyz="0 0 0" />
-  </joint>
-  <link name="camera_link">
-    <visual>
-      <origin xyz="0 0 0" rpy="0 0 0" />
-      <geometry>
-        <mesh filename="package://mobile_manipulator/meshes/base/camera.stl" />
-      </geometry>
-      <material name="">
-        <color rgba="0.79216 0.81961 0.93333 1" />
-      </material>
-    </visual>
-    <collision>
-      <origin xyz="0 0 0" rpy="0 0 0" />
-      <geometry>
-        <mesh filename="package://mobile_manipulator/meshes/base/camera.stl" />
-      </geometry>
-    </collision>
-    <xacro:inertial_cylinder mass="${camera_mass}" length="0.08832" radius="0.01265">
-      <origin xyz="0 0 0" rpy="-${M_PI/2} 0 0" />
-    </xacro:inertial_cylinder>
-  </link>
-  <joint name="base_arm_connector_joint" type="fixed">
-    <origin xyz="0 0 0.0576" rpy="0 0 0" />
-    <parent link="base_body" />
-    <child link="base_arm_connector"/>
-    <axis xyz="0 0 0" />
-  </joint>
-  <link name="base_arm_connector">
-    <visual>
-      <origin xyz="0 0 -0.0288" rpy="0 0 0" />
-      <geometry>
-        <mesh filename="package://mobile_manipulator/meshes/base/base_arm_connector.stl" />
-      </geometry>
-      <material name="">
-        <color rgba="0.79216 0.81961 0.93333 1" />
-      </material>
-    </visual>
-    <collision>
-      <origin xyz="0 0 -0.0288" rpy="0 0 0" />
-      <geometry>
-        <mesh filename="package://mobile_manipulator/meshes/base/base_arm_connector.stl" />
-      </geometry>
-    </collision>
-    <xacro:inertial_truncated_cone mass="${base_arm_connector_mass}" r1="0.03697" r2="0.05137" height="0.0576">
-      <origin xyz="0 0 -0.0288" rpy="0 0 0" />
-    </xacro:inertial_truncated_cone>
-  </link>
-  <gazebo reference="base_arm_connector">
-      <material>Kortex/Gray</material>
-  </gazebo>
+	<xacro:macro name="load_base" params="
+    parent">
+    <xacro:property name="M_PI" value="3.14159265358979323846" />
+    <xacro:property name="base_body_width" value="0.4" />
+    <xacro:property name="base_body_length" value="0.4" />
+    <xacro:property name="total_height" value="0.29386" />
+    <xacro:property name="front_wheel_length" value="0.127547" />
+    <xacro:property name="front_wheel_radius" value="0.0575" />
+    <xacro:property name="front_wheel_depth" value="0.079536242431022" />
+    <xacro:property name="rear_wheel_length" value="0.125" />
+    <xacro:property name="rear_wheel_radius" value="0.0325" />
+    <xacro:property name="rear_wheel_depth" value="0.022335230282742743" />
+    <!-- About the mass ratio of each part: -->
+    <xacro:property name="base_body_mass" value="24.3948952632956" />
+    <xacro:property name="front_wheel_mass" value="1.0568406891164" />
+    <xacro:property name="rear_wheel_bracket_mass" value="0.0211573699864" />
+    <xacro:property name="rear_wheel_mass" value="0.0920111896829" />
+    <xacro:property name="camera_mass" value="0.2333248928640" />
+    <xacro:property name="lidar_mass" value="0.1071556446529" />
+    <xacro:property name="base_arm_connector_mass" value="0.4535071053510" />
+    <!-- Include inertial xacro files -->
+    <xacro:include filename="$(find mobile_manipulator)/urdf/inertial.xacro" />
+    <joint name="base_body_joint" type="fixed">
+      <origin xyz="0 0 ${total_height}" rpy="0 0 0" />
+      <parent link="${parent}" />
+      <child link="base_body" />
+      <axis xyz="0 0 0" />
+    </joint>
+    <link name="base_body">
+      <visual>
+        <origin xyz="0 0 0" rpy="0 0 0" />
+        <geometry>
+          <mesh filename="package://mobile_manipulator/meshes/base/base_body.stl" />
+        </geometry>
+        <material name="">
+          <color rgba="1 1 1 1" />
+        </material>
+      </visual>
+      <collision>
+        <origin xyz="0 0 0" rpy="0 0 0" />
+        <geometry>
+          <mesh filename="package://mobile_manipulator/meshes/base/base_body.stl" />
+        </geometry>
+      </collision>
+      <xacro:inertial_box mass="${base_body_mass}" x="0.4" y="0.4" z="0.26344">
+        <origin xyz="0 0 0" rpy="0 0 0" />
+      </xacro:inertial_box>
+    </link>
+    <joint name="fl_joint" type="continuous">
+      <origin xyz="0.05 ${front_wheel_length} ${front_wheel_radius - total_height} " rpy="-${M_PI / 2} 0 0"/>
+      <parent link="base_body" />
+      <child link="fl_wheel" />
+      <axis xyz="0 0 1" />
+    </joint>
+    <link name="fl_wheel">
+      <visual>
+        <origin rpy="${M_PI/2} 0 0" xyz="0 0 0" />
+        <geometry>
+          <mesh filename="package://mobile_manipulator/meshes/base/front_wheel.stl" />
+        </geometry>
+        <material name="">
+          <color rgba="0.5 0.5 0.5 1" />
+        </material>
+      </visual>
+      <collision>
+        <origin rpy="${M_PI/2} 0 0" xyz="0 0 0" />
+        <geometry>
+          <mesh filename="package://mobile_manipulator/meshes/base/front_wheel.stl" />
+        </geometry>
+      </collision>
+      <xacro:inertial_cylinder mass="${front_wheel_mass}" length="${front_wheel_depth}" radius="${front_wheel_radius}">
+        <origin rpy="${M_PI/2} 0 0" xyz="0 0 0" />
+      </xacro:inertial_cylinder>
+    </link>
+    <joint name="fr_joint" type="continuous">
+      <origin xyz="0.05 -${front_wheel_length} ${front_wheel_radius - total_height}" rpy="${M_PI/2} 0 0" />
+      <parent link="base_body" />
+      <child link="fr_wheel" />
+      <axis xyz="0 0 1" />
+    </joint>
+    <link name="fr_wheel">
+      <visual>
+        <origin rpy="-${M_PI/2} 0 0" xyz="0 0 0" />
+        <geometry>
+          <mesh filename="package://mobile_manipulator/meshes/base/front_wheel.stl" />
+        </geometry>
+        <material name="">
+          <color rgba="0.5 0.5 0.5 1" />
+        </material>
+      </visual>
+      <collision>
+        <origin rpy="-${M_PI/2} 0 0" xyz="0 0 0" />
+        <geometry>
+          <mesh filename="package://mobile_manipulator/meshes/base/front_wheel.stl" />
+        </geometry>
+      </collision>
+      <xacro:inertial_cylinder mass="${front_wheel_mass}" length="${front_wheel_depth}" radius="${front_wheel_radius}">
+        <origin rpy="-${M_PI/2} 0 0" xyz="0 0 0" />
+      </xacro:inertial_cylinder>
+    </link>
+    <joint name="rl_bracket_joint" type="continuous">
+      <origin xyz="-0.17043 ${rear_wheel_length} ${rear_wheel_radius - total_height + 0.0453}" rpy="0 0 0" />
+      <parent link="base_body" />
+      <child link="rl_bracket" />
+      <axis xyz="0 0 1" />
+    </joint>
+    <link name="rl_bracket">
+      <visual>
+        <origin rpy="0 0 ${M_PI/2}" xyz="0 0 0" />
+        <geometry>
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
File: mobile_manipulator/urdf/execution.urdf.xacro (robot description, xacro)
@@ -3,5 +3,5 @@
     <xacro:arg name="name" default="mobile_manipulator"/>
     <!-- Arguments -->
-    <xacro:arg name="prefix" default="arm"/>
+    <xacro:arg name="robot_type" default=""/>
     <xacro:arg name="arm" default="gen3_lite"/>
     <xacro:arg name="dof" default="6"/>
@@ -30,5 +30,7 @@
     <xacro:arg name="initial_positions_file" default="$(find mobile_manipulator)/config/initial_positions.yaml"/>
     <xacro:property name="initial_positions_file" default="$(arg initial_positions_file)"/>
+    <link name="base_link"/>
     <xacro:load_robot
+        robot_type="$(arg robot_type)"
         vision="$(arg vision)"
         robot_ip="$(arg robot_ip)"

File: mobile_manipulator/urdf/execution.xacro (robot description, xacro)
@@ -2,4 +2,5 @@
 <robot xmlns:xacro="http://ros.org/wiki/xacro">
 	<xacro:macro name="load_robot" params="
+    robot_type
     vision
     robot_ip
@@ -24,34 +25,74 @@
     initial_positions:=${dict(joint_1=0.0,joint_2=0.0,joint_3=0.0,joint_4=0.0,joint_5=0.0,joint_6=0.0)}
     gripper_com_port:=/dev/ttyUSB0">
-		<!-- Include arm macro files -->
-		<!-- <xacro:include filename="$(find mobile_manipulator)/urdf/arm_and_gripper.xacro" /> -->
-    <xacro:include filename="$(find mobile_manipulator)/urdf/base.xacro" />
-    <xacro:include filename="$(find mobile_manipulator)/urdf/integrated_model.xacro" />
-		<!-- Load the arm -->
-    <xacro:load_arm
-      parent="${connection_link}"
-      vision="${vision}"
-      robot_ip="${robot_ip}"
-      username="${username}"
-      password="${password}"
-      port="${port}"
-      port_realtime="${port_realtime}"
-      session_inactivity_timeout_ms="${session_inactivity_timeout_ms}"
-      connection_inactivity_timeout_ms="${connection_inactivity_timeout_ms}"
-      use_internal_bus_gripper_comm="${use_internal_bus_gripper_comm}"
-      use_fake_hardware="${use_fake_hardware}"
-      fake_sensor_commands="${fake_sensor_commands}"
-      sim_gazebo="${sim_gazebo}"
-      sim_ignition="${sim_ignition}"
-      sim_isaac="${sim_isaac}"
-      isaac_joint_commands="${isaac_joint_commands}"
-      isaac_joint_states="${isaac_joint_states}"
-      gripper_joint_name="${gripper_joint_name}"
-      gripper_max_velocity="${gripper_max_velocity}"
-      gripper_max_force="${gripper_max_force}"
-      use_external_cable="${use_external_cable}"
-      initial_positions="${initial_positions}"
-			gripper_com_port="${gripper_com_port}">
-    </xacro:load_arm>
+    <!-- if robot_type is base, load the base.xacro file -->
+    <xacro:if value="${robot_type == 'base'}">
+      <xacro:include filename="$(find mobile_manipulator)/urdf/${robot_type}.xacro" />
+      <xacro:load_base
+        parent="base_link">
+      </xacro:load_base>
+    </xacro:if>
+    <!-- if robot_type is arm, load the arm.xacro file -->
+    <xacro:if value="${robot_type == 'arm'}">
+      <xacro:include filename="$(find mobile_manipulator)/urdf/${robot_type}.xacro" />
+      <xacro:load_arm
+        parent="base_link"
+        vision="${vision}"
+        robot_ip="${robot_ip}"
+        username="${username}"
+        password="${password}"
+        port="${port}"
+        port_realtime="${port_realtime}"
+        session_inactivity_timeout_ms="${session_inactivity_timeout_ms}"
+        connection_inactivity_timeout_ms="${connection_inactivity_timeout_ms}"
+        use_internal_bus_gripper_comm="${use_internal_bus_gripper_comm}"
+        use_fake_hardware="${use_fake_hardware}"
+        fake_sensor_commands="${fake_sensor_commands}"
+        sim_gazebo="${sim_gazebo}"
+        sim_ignition="${sim_ignition}"
+        sim_isaac="${sim_isaac}"
+        isaac_joint_commands="${isaac_joint_commands}"
+        isaac_joint_states="${isaac_joint_states}"
+        gripper_joint_name="${gripper_joint_name}"
+        gripper_max_velocity="${gripper_max_velocity}"
+        gripper_max_force="${gripper_max_force}"
+        use_external_cable="${use_external_cable}"
+        initial_positions="${initial_positions}"
+        gripper_com_port="${gripper_com_port}">
+      </xacro:load_arm>
+    </xacro:if>
+    <!-- if robot_type is integrate, load the integrated model with base and arm -->
+    <xacro:if value="${robot_type == 'integrate'}">
+      <xacro:include filename="$(find mobile_manipulator)/urdf/base.xacro" />
+      <xacro:load_base
+        parent="base_link">
+      </xacro:load_base>
+      <xacro:include filename="$(find mobile_manipulator)/urdf/integrated_model.xacro" />
+      <xacro:load_arm
+        parent="${connection_link}"
+        vision="${vision}"
+        robot_ip="${robot_ip}"
+        username="${username}"
+        password="${password}"
+        port="${port}"
+        port_realtime="${port_realtime}"
+        session_inactivity_timeout_ms="${session_inactivity_timeout_ms}"
+        connection_inactivity_timeout_ms="${connection_inactivity_timeout_ms}"
+        use_internal_bus_gripper_comm="${use_internal_bus_gripper_comm}"
+        use_fake_hardware="${use_fake_hardware}"
+        fake_sensor_commands="${fake_sensor_commands}"
+        sim_gazebo="${sim_gazebo}"
+        sim_ignition="${sim_ignition}"
+        sim_isaac="${sim_isaac}"
+        isaac_joint_commands="${isaac_joint_commands}"
+        isaac_joint_states="${isaac_joint_states}"
+        gripper_joint_name="${gripper_joint_name}"
+        gripper_max_velocity="${gripper_max_velocity}"
+        gripper_max_force="${gripper_max_force}"
+        use_external_cable="${use_external_cable}"
+        initial_positions="${initial_positions}"
+        gripper_com_port="${gripper_com_port}">
+      </xacro:load_arm>
+    </xacro:if>
+		<!-- Include xacro files -->
 	</xacro:macro>
 </robot>
