Commit message: 0925

File: mobile_manipulator/urdf/arm.xacro (robot description, xacro)
@@ -5,24 +5,23 @@
     vision
     robot_ip
-    username:=admin
-    password:=admin
-    port:=10000
-    port_realtime:=10001
-    session_inactivity_timeout_ms:=6000
-    connection_inactivity_timeout_ms:=2000
-    use_internal_bus_gripper_comm:=true
-    use_fake_hardware:=false
-    fake_sensor_commands:=false
-    sim_gazebo:=false
-    sim_ignition:=false
-    sim_isaac:=false
-    isaac_joint_commands:=/isaac_joint_commands
-    isaac_joint_states:=/isaac_joint_states
+    username
+    password
+    port
+    port_realtime
+    session_inactivity_timeout_ms
+    connection_inactivity_timeout_ms
+    use_internal_bus_gripper_comm:=/true
+    use_fake_hardware
+    fake_sensor_commands
+    sim_gazebo
+    sim_ignition
+    sim_isaac
+    isaac_joint_commands:=/arm_isaac_joint_commands
+    isaac_joint_states:=/arm_isaac_joint_states
     gripper_joint_name
-    gripper_max_velocity:=100.0
-    gripper_max_force:=100.0
-    use_external_cable:=false
-    initial_positions:=${dict(joint_1=0.0,joint_2=0.0,joint_3=0.0,joint_4=0.0,joint_5=0.0,joint_6=0.0)}
+    gripper_max_velocity
+    gripper_max_force
 		gripper_com_port">
+    <!-- arm and gripper xacro files -->
     <joint name="arm_base_joint" type="fixed">
       <origin xyz="0 0 0" rpy="0 0 0" />

File: mobile_manipulator/urdf/base.xacro (robot description, xacro)
@@ -2,26 +2,32 @@
 <robot name="tracer_mini" xmlns:xacro="http://www.ros.org/wiki/xacro">
   <xacro:property name="connection_link" value="base_arm_connector" />
+  <xacro:property name="M_PI" value="3.14159265358979323846" />
+  <xacro:property name="base_body_width" value="0.4" />
+  <xacro:property name="base_body_length" value="0.4" />
+  <xacro:property name="total_height" value="0.29386" />
+  <xacro:property name="front_wheel_length" value="0.127547" />
+  <xacro:property name="front_wheel_radius" value="0.0575" />
+  <xacro:property name="front_wheel_depth" value="0.079536242431022" />
+  <xacro:property name="rear_wheel_length" value="0.125" />
+  <xacro:property name="rear_wheel_radius" value="0.0325" />
+  <xacro:property name="rear_wheel_depth" value="0.022335230282742743" />
+  <!-- About the mass ratio of each part: -->
+  <xacro:property name="base_body_mass" value="24.3948952632956" />
+  <xacro:property name="front_wheel_mass" value="1.0568406891164" />
+  <xacro:property name="rear_wheel_bracket_mass" value="0.0211573699864" />
+  <xacro:property name="rear_wheel_mass" value="0.0920111896829" />
+  <xacro:property name="camera_mass" value="0.2333248928640" />
+  <xacro:property name="lidar_mass" value="0.1071556446529" />
+  <xacro:property name="base_arm_connector_mass" value="0.4535071053510" />
+  <xacro:include filename="$(find mobile_manipulator)/urdf/inertial.xacro" />
 	<xacro:macro name="load_base" params="
-    parent">
-    <xacro:property name="M_PI" value="3.14159265358979323846" />
-    <xacro:property name="base_body_width" value="0.4" />
-    <xacro:property name="base_body_length" value="0.4" />
-    <xacro:property name="total_height" value="0.29386" />
-    <xacro:property name="front_wheel_length" value="0.127547" />
-    <xacro:property name="front_wheel_radius" value="0.0575" />
-    <xacro:property name="front_wheel_depth" value="0.079536242431022" />
-    <xacro:property name="rear_wheel_length" value="0.125" />
-    <xacro:property name="rear_wheel_radius" value="0.0325" />
-    <xacro:property name="rear_wheel_depth" value="0.022335230282742743" />
-    <!-- About the mass ratio of each part: -->
-    <xacro:property name="base_body_mass" value="24.3948952632956" />
-    <xacro:property name="front_wheel_mass" value="1.0568406891164" />
-    <xacro:property name="rear_wheel_bracket_mass" value="0.0211573699864" />
-    <xacro:property name="rear_wheel_mass" value="0.0920111896829" />
-    <xacro:property name="camera_mass" value="0.2333248928640" />
-    <xacro:property name="lidar_mass" value="0.1071556446529" />
-    <xacro:property name="base_arm_connector_mass" value="0.4535071053510" />
-    <!-- Include inertial xacro files -->
-    <xacro:include filename="$(find mobile_manipulator)/urdf/inertial.xacro" />
+    parent
+    use_fake_hardware
+    fake_sensor_commands
+    sim_gazebo
+    sim_ignition
+    sim_isaac
+    isaac_joint_commands:=/base_isaac_joint_commands
+    isaac_joint_states:=/base_isaac_joint_states">
     <joint name="base_body_joint" type="fixed">
       <origin xyz="0 0 ${total_height}" rpy="0 0 0" />
@@ -55,4 +61,5 @@
       <child link="fl_wheel" />
       <axis xyz="0 0 1" />
+      <dynamics damping="0.1" friction="0.1" />
     </joint>
     <link name="fl_wheel">
@@ -81,4 +88,5 @@
       <child link="fr_wheel" />
       <axis xyz="0 0 1" />
+      <dynamics damping="0.1" friction="0.1" />
     </joint>
     <link name="fr_wheel">
@@ -107,4 +115,5 @@
       <child link="rl_bracket" />
       <axis xyz="0 0 1" />
+      <dynamics damping="0.1" friction="0.0" />
     </joint>
     <link name="rl_bracket">
@@ -133,4 +142,5 @@
       <child link="rl_wheel" />
       <axis xyz="0 0 1" />
+      <dynamics damping="0.1" friction="0.0" />
     </joint>
     <link name="rl_wheel">
@@ -154,9 +164,10 @@
       </xacro:inertial_cylinder>
     </link>
-    <joint name="rr_bracekt_joint" type="continuous">
+    <joint name="rr_bracket_joint" type="continuous">
       <origin xyz="-0.17043 -${rear_wheel_length} ${rear_wheel_radius - total_height + 0.0453}" rpy="0 0 0" />
       <parent link="base_body" />
       <child link="rr_bracket" />
       <axis xyz="0 0 1" />
+      <dynamics damping="0.1" friction="0.0" />
     </joint>
     <link name="rr_bracket">
@@ -185,4 +196,5 @@
       <child link="rr_wheel" />
       <axis xyz="0 0 1" />
+      <dynamics damping="0.1" friction="0.0" />
     </joint>
     <link name="rr_wheel">

File: mobile_manipulator/urdf/view.xacro (robot description, xacro)
@@ -11,24 +11,30 @@
     session_inactivity_timeout_ms
     connection_inactivity_timeout_ms
-    use_internal_bus_gripper_comm:=false
-    use_fake_hardware:=false
-    fake_sensor_commands:=false
-    sim_gazebo:=false
-    sim_ignition:=false
-    sim_isaac:=false
-    isaac_joint_commands:=/isaac_joint_commands
-    isaac_joint_states:=/isaac_joint_states
+    use_internal_bus_gripper_comm
+    use_fake_hardware
+    fake_sensor_commands
+    sim_gazebo
+    sim_ignition
+    sim_isaac
     gripper_joint_name
-    gripper_max_velocity:=100.0
-    gripper_max_force:=100.0
-    use_external_cable:=false
-    initial_positions:=${dict(joint_1=0.0,joint_2=0.0,joint_3=0.0,joint_4=0.0,joint_5=0.0,joint_6=0.0)}
+    gripper_max_velocity
+    gripper_max_force
     gripper_com_port:=/dev/ttyUSB0">
+    <xacro:arg name="base_isaac_joint_commands" default="/base_isaac_joint_commands"/>
+    <xacro:arg name="base_isaac_joint_states" default="/base_isaac_joint_states"/>
+    <xacro:arg name="arm_isaac_joint_commands" default="/arm_isaac_joint_commands"/>
+    <xacro:arg name="arm_isaac_joint_states" default="/arm_isaac_joint_states"/>
     <!-- if robot_type is base, load the base.xacro file -->
     <xacro:if value="${robot_type == 'base'}">
       <xacro:include filename="$(find mobile_manipulator)/urdf/${robot_type}.xacro" />
       <xacro:load_base
-        parent="base_link">
-      </xacro:load_base>
+        parent="base_link"
+        use_fake_hardware="${use_fake_hardware}"
+        fake_sensor_commands="${fake_sensor_commands}"
+        sim_gazebo="${sim_gazebo}"
+        sim_ignition="${sim_ignition}"
+        sim_isaac="${sim_isaac}"
+        isaac_joint_commands="$(arg base_isaac_joint_commands)"
+        isaac_joint_states="$(arg base_isaac_joint_states)"/>
     </xacro:if>
     <!-- if robot_type is arm, load the arm.xacro file -->
@@ -51,21 +57,24 @@
         sim_ignition="${sim_ignition}"
         sim_isaac="${sim_isaac}"
-        isaac_joint_commands="${isaac_joint_commands}"
-        isaac_joint_states="${isaac_joint_states}"
+        isaac_joint_commands="$(arg arm_isaac_joint_commands)"
+        isaac_joint_states="$(arg arm_isaac_joint_states)"
         gripper_joint_name="${gripper_joint_name}"
         gripper_max_velocity="${gripper_max_velocity}"
         gripper_max_force="${gripper_max_force}"
-        use_external_cable="${use_external_cable}"
-        initial_positions="${initial_positions}"
-        gripper_com_port="${gripper_com_port}">
-      </xacro:load_arm>
+        gripper_com_port="${gripper_com_port}"/>
     </xacro:if>
     <!-- if robot_type is integrate, load the integrated model with base and arm -->
     <xacro:if value="${robot_type == 'integrate'}">
       <xacro:include filename="$(find mobile_manipulator)/urdf/base.xacro" />
+      <xacro:include filename="$(find mobile_manipulator)/urdf/arm.xacro" />
       <xacro:load_base
-        parent="base_link">
-      </xacro:load_base>
-      <xacro:include filename="$(find mobile_manipulator)/urdf/integrated_model.xacro" />
+        parent="base_link"
+        use_fake_hardware="${use_fake_hardware}"
+        fake_sensor_commands="${fake_sensor_commands}"
+        sim_gazebo="${sim_gazebo}"
+        sim_ignition="${sim_ignition}"
+        sim_isaac="${sim_isaac}"
+        isaac_joint_commands="$(arg base_isaac_joint_commands)"
+        isaac_joint_states="$(arg base_isaac_joint_states)"/>
       <xacro:load_arm
         parent="${connection_link}"
@@ -84,15 +93,11 @@
         sim_ignition="${sim_ignition}"
         sim_isaac="${sim_isaac}"
-        isaac_joint_commands="${isaac_joint_commands}"
-        isaac_joint_states="${isaac_joint_states}"
+        isaac_joint_commands="$(arg arm_isaac_joint_commands)"
+        isaac_joint_states="$(arg arm_isaac_joint_states)"
         gripper_joint_name="${gripper_joint_name}"
         gripper_max_velocity="${gripper_max_velocity}"
         gripper_max_force="${gripper_max_force}"
-        use_external_cable="${use_external_cable}"
-        initial_positions="${initial_positions}"
-        gripper_com_port="${gripper_com_port}">
-      </xacro:load_arm>
+        gripper_com_port="${gripper_com_port}"/>
     </xacro:if>
-		<!-- Include xacro files -->
 	</xacro:macro>
 </robot>
