Commit message: 1010

File: mobile_manipulator/urdf/integrate_ros2_control.xacro (robot description, xacro)
@@ -10,6 +10,9 @@
     isaac_joint_states
     initial_value">
-    <ros2_control name="ros2_control" type="system">
+    <ros2_control name="HC_control" type="system">
       <hardware>
+        <xacro:if value="${sim_ignition}">
+          <plugin>ign_ros2_control/IgnitionSystem</plugin>
+        </xacro:if>
         <xacro:if value="${sim_gazebo}">
           <plugin>gazebo_ros2_control/GazeboSystem</plugin>
@@ -28,6 +31,7 @@
       <joint name="fl_joint">
         <command_interface name="velocity"/>
-        <state_interface name="position"/>
+        <state_interface name="position">
           <param name="initial_value">${initial_value['fl_joint']}</param>
+        </state_interface>
         <state_interface name="velocity"/>
         <state_interface name="effort"/>
@@ -35,6 +39,7 @@
       <joint name="fr_joint">
         <command_interface name="velocity"/>
-        <state_interface name="position"/>
+        <state_interface name="position">
           <param name="initial_value">${initial_value['fr_joint']}</param>
+        </state_interface>
         <state_interface name="velocity"/>
         <state_interface name="effort"/>
@@ -145,34 +150,162 @@
         <state_interface name="effort"/>
       </joint>
-      <xacro:if value="${use_fake_hardware or sim_isaac}">
+      <xacro:if value="${use_fake_hardware or sim_isaac or sim_ignition}">
         <joint name="right_finger_tip_joint">
           <param name="mimic">right_finger_bottom_joint</param>
           <param name="multiplier">-1.0</param>
-          <command_interface name="position"/>
-          <state_interface name="position"/>
-            <param name="initial_value">${initial_value['right_finger_tip_joint']}</param>
-          <state_interface name="velocity"/>
-          <state_interface name="effort"/>
+          <xacro:unless value="${sim_ignition}">
+            <command_interface name="position"/>
+            <state_interface name="position"/>
+            <state_interface name="velocity"/>
+            <state_interface name="effort"/>
+          </xacro:unless>
         </joint>
         <joint name="left_finger_bottom_joint">
           <param name="mimic">right_finger_bottom_joint</param>
           <param name="multiplier">1.0</param>
-          <command_interface name="position"/>
-          <state_interface name="position"/>
-            <param name="initial_value">${initial_value['left_finger_bottom_joint']}</param>
-          <state_interface name="velocity"/>
-          <state_interface name="effort"/>
+          <xacro:unless value="${sim_ignition}">
+            <command_interface name="position"/>
+            <state_interface name="position"/>
+            <state_interface name="velocity"/>
+            <state_interface name="effort"/>
+          </xacro:unless>
         </joint>
         <joint name="left_finger_tip_joint">
           <param name="mimic">right_finger_bottom_joint</param>
           <param name="multiplier">-1.0</param>
-          <command_interface name="position"/>
-          <state_interface name="position"/>
-            <param name="initial_value">${initial_value['left_finger_tip_joint']}</param>
-          <state_interface name="velocity"/>
-          <state_interface name="effort"/>
+          <xacro:unless value="${sim_ignition}">
+            <command_interface name="position"/>
+            <state_interface name="position"/>
+            <state_interface name="velocity"/>
+            <state_interface name="effort"/>
+          </xacro:unless>
         </joint>
       </xacro:if>
     </ros2_control>
+    <transmission name="fl_joint_transmission">
+      <type>transmission_interface/SimpleTransmission</type>
+      <joint name="fl_joint">
+        <hardwareInterface>hardware_interface/VelocityJointInterface</hardwareInterface>
+      </joint>
+      <actuator name="fl_wheel_motor">
+        <mechanicalReduction>1</mechanicalReduction>
+      </actuator>
+    </transmission>
+    <transmission name="fr_joint_transmission">
+      <type>transmission_interface/SimpleTransmission</type>
+      <joint name="fr_joint">
+        <hardwareInterface>hardware_interface/VelocityJointInterface</hardwareInterface>
+      </joint>
+      <actuator name="fr_wheel_motor">
+        <mechanicalReduction>1</mechanicalReduction>
+      </actuator>
+    </transmission>
+    <transmission name="arm_joint_1_transmission">
+      <type>transmission_interface/SimpleTransmission</type>
+      <joint name="arm_joint_1">
+        <hardwareInterface>hardware_interface/PositionJointInterface</hardwareInterface>
+      </joint>
+      <actuator name="arm_joint_1_motor">
+        <mechanicalReduction>1</mechanicalReduction>
+      </actuator>
+    </transmission>
+    <transmission name="arm_joint_2_transmission">
+      <type>transmission_interface/SimpleTransmission</type>
+      <joint name="arm_joint_2">
+        <hardwareInterface>hardware_interface/PositionJointInterface</hardwareInterface>
+      </joint>
+      <actuator name="arm_joint_2_motor">
+        <mechanicalReduction>1</mechanicalReduction>
+      </actuator>
+    </transmission>
+    <transmission name="arm_joint_3_transmission">
+      <type>transmission_interface/SimpleTransmission</type>
+      <joint name="arm_joint_3">
+        <hardwareInterface>hardware_interface/PositionJointInterface</hardwareInterface>
+      </joint>
+      <actuator name="arm_joint_3_motor">
+        <mechanicalReduction>1</mechanicalReduction>
+      </actuator>
+    </transmission>
+    <transmission name="arm_joint_4_transmission">
+      <type>transmission_interface/SimpleTransmission</type>
+      <joint name="arm_joint_4">
+        <hardwareInterface>hardware_interface/PositionJointInterface</hardwareInterface>
+      </joint>
+      <actuator name="arm_joint_4_motor">
+        <mechanicalReduction>1</mechanicalReduction>
+      </actuator>
+    </transmission>
+    <transmission name="arm_joint_5_transmission">
+      <type>transmission_interface/SimpleTransmission</type>
+      <joint name="arm_joint_5">
+        <hardwareInterface>hardware_interface/PositionJointInterface</hardwareInterface>
+      </joint>
+      <actuator name="arm_joint_5_motor">
+        <mechanicalReduction>1</mechanicalReduction>
+      </actuator>
+    </transmission>
+    <transmission name="arm_joint_6_transmission">
+      <type>transmission_interface/SimpleTransmission</type>
+      <joint name="arm_joint_6">
+        <hardwareInterface>hardware_interface/PositionJointInterface</hardwareInterface>
+      </joint>
+      <actuator name="arm_joint_6_motor">
+        <mechanicalReduction>1</mechanicalReduction>
+      </actuator>
+    </transmission>
+    <transmission name="right_finger_bottom_joint_transmission">
+      <type>transmission_interface/SimpleTransmission</type>
+      <joint name="right_finger_bottom_joint">
+        <hardwareInterface>hardware_interface/PositionJointInterface</hardwareInterface>
+      </joint>
+      <actuator name="right_finger_bottom_joint_motor">
+        <mechanicalReduction>1</mechanicalReduction>
+        <hardwareInterface>hardware_interface/PositionJointInterface</hardwareInterface>
+      </actuator>
+    </transmission>
+    <xacro:if value="${sim_gazebo}">
+      <gazebo>
+        <plugin filename="libroboticsgroup_gazebo_mimic_joint_plugin.so" name="mimic_right_finger_tip_joint">
+          <joint>right_finger_bottom_joint</joint>
+          <mimicJoint>right_finger_tip_joint</mimicJoint>
+          <multiplier>-0.676</multiplier>
+          <offset>0.149</offset>
+          <maxEffort>5.0</maxEffort>
+          <hasPID></hasPID>
+        </plugin>
+        <plugin filename="libroboticsgroup_gazebo_mimic_joint_plugin.so" name="mimic_left_finger_bottom_joint">
+          <joint>right_finger_bottom_joint</joint>
+          <mimicJoint>left_finger_bottom_joint</mimicJoint>
+          <multiplier>-1.0</multiplier>
+          <offset>0.0</offset>
+          <maxEffort>5.0</maxEffort>
+          <hasPID></hasPID>
+        </plugin>
+        <plugin filename="libroboticsgroup_gazebo_mimic_joint_plugin.so" name="mimic_left_finger_tip_joint">
+          <joint>right_finger_bottom_joint</joint>
+          <mimicJoint>left_finger_tip_joint</mimicJoint>
+          <multiplier>-0.676</multiplier>
+          <offset>0.149</offset>
+          <maxEffort>5.0</maxEffort>
+          <hasPID></hasPID>
+        </plugin>
+        <plugin filename="libgazebo_grasp_fix.so" name="gazebo_grasp_fix">
+          <arm>
+            <arm_name>mobile_manipulator_gripper</arm_name>
+            <palm_link>end_effector_link</palm_link>
+            <gripper_link>right_finger_dist_link</gripper_link>
+            <gripper_link>left_finger_dist_link</gripper_link>
+          </arm>
+          <forces_angle_tolerance>100</forces_angle_tolerance>
+          <update_rate>10</update_rate>
+          <grip_count_threshold>3</grip_count_threshold>
+          <max_grip_count>10</max_grip_count>
+          <release_tolerance>0.001</release_tolerance>
+          <disable_collisions_on_attach>false</disable_collisions_on_attach>
+          <contact_topic>__default_topic__</contact_topic>
+        </plugin>
+      </gazebo>
+    </xacro:if>
   </xacro:macro>
 </robot>
