Commit message: 0926

File: mobile_manipulator/urdf/integrate_execution.xacro (robot description, xacro)
@@ -20,6 +20,6 @@
 	<xacro:arg name="gazebo_renderer" default="ogre"/>
 	<xacro:arg name="gripper_com_port" default="/dev/ttyUSB0"/>
-	<xacro:arg name="issac_joint_commands" default="/isaac_joint_commands"/>
-	<xacro:arg name="issac_joint_states" default="/isaac_joint_states"/>
+	<xacro:arg name="isaac_joint_commands" default="/isaac_joint_commands"/>
+	<xacro:arg name="isaac_joint_states" default="/isaac_joint_states"/>
 	<xacro:arg name="simulation_controllers" default="$(find mobile_manipulator)/config/ros2_control.yaml"/>
 	<xacro:arg name="initial_value" default="$(find mobile_manipulator)/config/initial_value.yaml"/>
@@ -44,6 +44,6 @@
 		gripper_max_velocity="$(arg gripper_max_velocity)"
 		gripper_max_force="$(arg gripper_max_force)"
-		isaac_joint_commands="$(arg issac_joint_commands)"
-		isaac_joint_states="$(arg issac_joint_states)"
+		isaac_joint_commands="$(arg isaac_joint_commands)"
+		isaac_joint_states="$(arg isaac_joint_states)"
 		initial_value="${xacro.load_yaml(initial_value)}"/>
 	<xacro:if value="$(arg sim_gazebo)">

File: mobile_manipulator/urdf/integrate_model.xacro (robot description, xacro)
@@ -261,11 +261,11 @@
       </xacro:inertial_cylinder>
     </link>
-    <joint name="camera_joint" type="fixed">
+    <joint name="base_camera_joint" type="fixed">
       <origin xyz="0.115 0 -0.04565" rpy="0 0 0" />
       <parent link="base_body" />
-      <child link="camera_link" />
+      <child link="base_camera_link" />
       <axis xyz="0 0 0" />
     </joint>
-    <link name="camera_link">
+    <link name="base_camera_link">
       <visual>
         <origin xyz="0 0 0" rpy="0 0 0" />
@@ -515,10 +515,68 @@
     <link name="end_effector_link"/>
     <joint name="tool_frame_joint" type="fixed">
-        <origin xyz="0 0 0.130" rpy="0 0 1.57079632679" />
-        <parent link="end_effector_link" />
-        <child link="tool_frame" />
-        <axis xyz="0 0 0" />
+      <origin xyz="0 0 0.130" rpy="0 0 -1.5708" />
+      <parent link="end_effector_link" />
+      <child link="tool_frame" />
+      <axis xyz="0 0 0" />
     </joint>
     <link name="tool_frame"/>
+    <joint name="camera_case_joint" type="fixed">
+      <origin xyz="0 0 0.01794" rpy="0 -1.5708 0"/>
+      <parent link="end_effector_link" />
+      <child link="camera_case_link" />
+      <axis xyz="0 0 0" />
+    </joint>
+    <link name="camera_case_link">
+      <visual>
+        <origin xyz="-0.01254 0 0" rpy="0 0 0" />
+        <geometry>
+          <mesh filename="package://mobile_manipulator/meshes/gripper/camera_case.stl" />
+        </geometry>
+        <material name="">
+          <color rgba="0 0 0 1" />
+        </material>
+      </visual>
+      <collision>
+        <origin xyz="0 0 0" rpy="0 0 0" />
+        <geometry>
+          <mesh filename="package://mobile_manipulator/meshes/gripper/camera_case.stl" />
+        </geometry>
+      </collision>
+      <xacro:inertial_box mass="${camera_mass}" x="0.0672" y="0.1282" z="0.01254">
+        <origin xyz="0 0 -0.05153" rpy="0 0 0" />
+      </xacro:inertial_box>
+    </link>
+    <gazebo reference="camera_case_link">
+      <material>Kortex/Black</material>
+    </gazebo>
+    <joint name="gripper_camera_joint" type="fixed">
+      <origin xyz="0 0 0.08203" ryp=" 0 0" />
+      <parent link="camera_case_link" />
+      <child link="gripper_camera"/>
+      <axis xyz="0 0 0" />
+    </joint>
+    <link name="gripper_camera">
+      <visual>
+        <origin xyz="0.025 0 0" rpy="0 0 1.5708" />
+        <geometry>
+          <mesh filename="package://mobile_manipulator/meshes/gripper/D435.stl" />
+        </geometry>
+        <material name="">
+          <color rgba="0.803 0.824 0.820 1" />
+        </material>
+      </visual>
+      <collision>
+        <origin xyz="0.025 0 0" rpy="0 0 1.5708" />
+        <geometry>
+          <mesh filename="package://mobile_manipulator/meshes/gripper/D435.stl" />
+        </geometry>
+      </collision>
+      <xacro:inertial_cylinder mass="${camera_mass}" length="0.08832" radius="0.01265">
+        <origin xyz="0.025 0 0" rpy="0 0 1.5708" />
+      </xacro:inertial_cylinder>
+    </link>
+    <gazebo reference="gripper_camera">
+      <material>Kortex/Gray</material>
+    </gazebo>
 		<joint name="gripper_base_joint" type="fixed">
       <origin xyz="0 0 0" rpy="0 0 0" />
@@ -528,4 +586,19 @@
     </joint>
 		<link name="gripper_base_link">
+      <visual>
+        <origin xyz="0 0 0" rpy="0 0 0" />
+        <geometry>
+          <mesh filename="package://mobile_manipulator/meshes/gripper/gripper_base_link.STL" />
+        </geometry>
+        <material name="">
+          <color rgba="0.803 0.824 0.820 1" />
+        </material>
+      </visual>
+      <collision>
+        <origin xyz="0 0 0" rpy="0 0 0" />
+        <geometry>
+          <mesh filename="package://mobile_manipulator/meshes/gripper/gripper_base_link.STL" />
+        </geometry>
+      </collision>
       <inertial>
         <origin xyz="4.03E-06 1.08E-05 0.041397" rpy="0 0 0" />
@@ -533,19 +606,4 @@
         <inertia ixx="0.00011614" ixy="1E-08" ixz="4E-08" iyy="0.00010327" iyz="0" izz="9.707E-05" />
       </inertial>
-      <visual>
-        <origin xyz="0 0 0" rpy="0 0 0" />
-        <geometry>
-          <mesh filename="package://mobile_manipulator/meshes/gripper/gripper_base_link.STL" />
-        </geometry>
-        <material name="">
-          <color rgba="0.803 0.824 0.820 1" />
-        </material>
-      </visual>
-      <collision>
-        <origin xyz="0 0 0" rpy="0 0 0" />
-        <geometry>
-          <mesh filename="package://mobile_manipulator/meshes/gripper/gripper_base_link.STL" />
-        </geometry>
-      </collision>
     </link>
     <gazebo reference="gripper_base_link">
@@ -560,4 +618,19 @@
     </joint>
     <link name="right_finger_prox_link">
+      <visual>
+        <origin xyz="0 0 0" rpy="0 0 0" />
+        <geometry>
+          <mesh filename="package://mobile_manipulator/meshes/gripper/right_finger_prox_link.STL" />
+        </geometry>
+        <material name="">
+            <color rgba="0.803 0.824 0.820 1" />
+        </material>
+      </visual>
+      <collision>
+        <origin xyz="0 0 0" rpy="0 0 0" />
+        <geometry>
+          <mesh filename="package://mobile_manipulator/meshes/gripper/right_finger_prox_link.STL" />
+        </geometry>
+      </collision>
       <inertial>
         <origin xyz="0.020257 0.0063483 6.991E-05" rpy="0 0 0" />
@@ -565,19 +638,4 @@
         <inertia ixx="2.29E-06" ixy="1.43E-06" ixz="0" iyy="4.56E-06" iyz="0" izz="4.77E-06" />
       </inertial>
-      <visual>
-        <origin xyz="0 0 0" rpy="0 0 0" />
-        <geometry>
-          <mesh filename="package://mobile_manipulator/meshes/gripper/right_finger_prox_link.STL" />
-        </geometry>
-        <material name="">
-            <color rgba="0.803 0.824 0.820 1" />
-        </material>
-      </visual>
-      <collision>
-        <origin xyz="0 0 0" rpy="0 0 0" />
-        <geometry>
-          <mesh filename="package://mobile_manipulator/meshes/gripper/right_finger_prox_link.STL" />
-        </geometry>
-      </collision>
     </link>
     <gazebo reference="right_finger_prox_link">
@@ -593,4 +651,19 @@
     </joint>
     <link name="right_finger_dist_link">
+      <visual>
+        <origin xyz="0 0 0" rpy="0 0 0" />
+        <geometry>
+          <mesh filename="package://mobile_manipulator/meshes/gripper/right_finger_dist_link.STL" />
+        </geometry>
+        <material name="">
+          <color rgba="0 0.055 0.525 1" />
+        </material>
+      </visual>
+      <collision>
+        <origin xyz="0 0 0" rpy="0 0 0" />
+        <geometry>
+          <mesh filename="package://mobile_manipulator/meshes/gripper/right_finger_dist_link.STL" />
+        </geometry>
+      </collision>
       <inertial>
         <origin xyz="0.018488 0.0011091 0" rpy="0 0 0" />
@@ -598,19 +671,4 @@
         <inertia ixx="6.3E-07" ixy="3.2E-07" ixz="0" iyy="1.83E-06" iyz="0" izz="1.61E-06" />
       </inertial>
-      <visual>
-        <origin xyz="0 0 0" rpy="0 0 0" />
-        <geometry>
-          <mesh filename="package://mobile_manipulator/meshes/gripper/right_finger_dist_link.STL" />
-        </geometry>
-        <material name="">
-          <color rgba="0 0.055 0.525 1" />
-        </material>
-      </visual>
-      <collision>
-        <origin xyz="0 0 0" rpy="0 0 0" />
-        <geometry>
-          <mesh filename="package://mobile_manipulator/meshes/gripper/right_finger_dist_link.STL" />
-        </geometry>
-      </collision>
     </link>
     <gazebo reference="right_finger_dist_link">
@@ -626,4 +684,19 @@
     </joint>
     <link name="left_finger_prox_link">
+      <visual>
+        <origin xyz="0 0 0" rpy="0 0 0" />
+        <geometry>
+          <mesh filename="package://mobile_manipulator/meshes/gripper/left_finger_prox_link.STL" />
+        </geometry>
+        <material name="">
+          <color rgba="0.803 0.824 0.820 1" />
+        </material>
+      </visual>
+      <collision>
+        <origin xyz="0 0 0" rpy="0 0 0" />
+        <geometry>
+          <mesh filename="package://mobile_manipulator/meshes/gripper/left_finger_prox_link.STL" />
+        </geometry>
+      </collision>
       <inertial>
         <origin xyz="0.020257 0.0063483 6.99E-05" rpy="0 0 0" />
@@ -631,19 +704,4 @@
         <inertia ixx="2.29E-06" ixy="1.43E-06" ixz="0" iyy="4.56E-06" iyz="0" izz="4.77E-06" />
       </inertial>
-      <visual>
-        <origin xyz="0 0 0" rpy="0 0 0" />
-        <geometry>
-          <mesh filename="package://mobile_manipulator/meshes/gripper/left_finger_prox_link.STL" />
-        </geometry>
-        <material name="">
-          <color rgba="0.803 0.824 0.820 1" />
-        </material>
-      </visual>
-      <collision>
-        <origin xyz="0 0 0" rpy="0 0 0" />
-        <geometry>
-          <mesh filename="package://mobile_manipulator/meshes/gripper/left_finger_prox_link.STL" />
-        </geometry>
-      </collision>
     </link>
     <gazebo reference="left_finger_prox_link">
@@ -659,4 +717,19 @@
     </joint>
     <link name="left_finger_dist_link">
+      <visual>
+        <origin xyz="0 0 0" rpy="0 0 0" />
+        <geometry>
+          <mesh filename="package://mobile_manipulator/meshes/gripper/left_finger_dist_link.STL" />
+        </geometry>
+        <material name="">
+          <color rgba="0 0.055 0.525 1" />
+        </material>
+      </visual>
+      <collision>
+        <origin xyz="0 0 0" rpy="0 0 0" />
+        <geometry>
+          <mesh filename="package://mobile_manipulator/meshes/gripper/left_finger_dist_link.STL" />
+        </geometry>
+      </collision>
       <inertial>
         <origin xyz="-0.018488 0.0011091 0" rpy="0 0 0" />
@@ -664,19 +737,4 @@
         <inertia ixx="6.3E-07" ixy="3.2E-07" ixz="0" iyy="1.83E-06" iyz="0" izz="1.61E-06" />
       </inertial>
-      <visual>
-        <origin xyz="0 0 0" rpy="0 0 0" />
-        <geometry>
-          <mesh filename="package://mobile_manipulator/meshes/gripper/left_finger_dist_link.STL" />
-        </geometry>
-        <material name="">
-          <color rgba="0 0.055 0.525 1" />
-        </material>
-      </visual>
-      <collision>
-        <origin xyz="0 0 0" rpy="0 0 0" />
-        <geometry>
-          <mesh filename="package://mobile_manipulator/meshes/gripper/left_finger_dist_link.STL" />
-        </geometry>
-      </collision>
     </link>
     <gazebo reference="left_finger_dist_link">

Commit message: 1010

File: mobile_manipulator/urdf/integrate_execution.xacro (robot description, xacro)
@@ -10,13 +10,13 @@
 	<xacro:arg name="connection_inactivity_timeout_ms" default="2000"/>
 	<xacro:arg name="use_internal_bus_gripper_comm" default="false"/>
-	<xacro:arg name="use_fake_hardware" default="true"/>
+	<xacro:arg name="use_fake_hardware" default="false"/>
 	<xacro:arg name="fake_sensor_commands" default="false"/>
 	<xacro:arg name="sim_gazebo" default="false"/>
-	<xacro:arg name="sim_ignition" default="false"/>
+	<xacro:arg name="sim_ignition" default="true"/>
 	<xacro:arg name="sim_isaac" default="false"/>
 	<xacro:arg name="gripper_joint_name" default="right_finger_bottom_joint"/>
 	<xacro:arg name="gripper_max_velocity" default="100.0"/>
 	<xacro:arg name="gripper_max_force" default="100.0"/>
-	<xacro:arg name="gazebo_renderer" default="ogre"/>
+	<xacro:arg name="gazebo_renderer" default="ogre2"/>
 	<xacro:arg name="gripper_com_port" default="/dev/ttyUSB0"/>
 	<xacro:arg name="isaac_joint_commands" default="/isaac_joint_commands"/>
@@ -25,5 +25,13 @@
 	<xacro:arg name="initial_value" default="$(find mobile_manipulator)/config/initial_value.yaml"/>
 	<xacro:property name="initial_value" default="$(arg initial_value)"/>
+  <xacro:property name="camera_width" value="1280"/>
+  <xacro:property name="camera_height" value="720"/>
+  <xacro:property name="camera_fps" value="30"/>
+  <xacro:property name="M_PI" value="3.1415926535897931" />
+  <xacro:property name="horizontal_fov" value="${69.4 * M_PI / 180}"/>
 	<xacro:include filename="$(find mobile_manipulator)/urdf/integrate_model.xacro"/>
+	<xacro:if value="$(arg sim_gazebo)">
+		<xacro:include filename="$(find mobile_manipulator)/urdf/integrate_gazebo.xacro"/>
+	</xacro:if>
 	<xacro:load_model
 		vision="$(arg vision)"
@@ -48,84 +56,24 @@
 		initial_value="${xacro.load_yaml(initial_value)}"/>
 	<xacro:if value="$(arg sim_gazebo)">
-		<gazebo reference="base_link"/>
+		<gazebo reference="world"/>
 		<gazebo>
-			<plugin filename="libgazebo_ros2_control.so" name="gazebo_ros2_control">
-					<parameters>$(arg simulation_controllers)</parameters>
+			<plugin filename="libgazebo_ros2_control-system.so" name="gazebo_ros2_control::GazeboROS2ControlPlugin">
+				<parameters>$(arg simulation_controllers)</parameters>
+				<controller_manager_node_name>controller_manager</controller_manager_node_name>
+			</plugin>
+			<plugin filename="libgazebo_ros_control_mimic_joint_plugin.so" name="mimic_joint_plugin"/>
+		</gazebo>
+	</xacro:if>
+	<xacro:if value="$(arg sim_ignition)">
+    <gazebo>
+			<plugin filename="libign_ros2_control-system.so" name="ign_ros2_control::IgnitionROS2ControlPlugin">
+				<namespace>/</namespace>
+				<parameters>$(arg simulation_controllers)</parameters>
+				<controller_manager_node_name>controller_manager</controller_manager_node_name>
+			</plugin>
+			<plugin filename="libignition-gazebo-sensors-system.so" name="ignition::gazebo::systems::Sensors">
+				<render_engine>$(arg gazebo_renderer)</render_engine>
 			</plugin>
 		</gazebo>
 	</xacro:if>
-	<xacro:if value="$(arg sim_ignition)">
-		<!-- Gazebo plugins -->
-		<gazebo reference="world"/>
-		<gazebo>
-			<plugin filename="libign_ros2_control-system.so" name="ign_ros2_control::IgnitionROS2ControlPlugin">
-					<parameters>$(arg simulation_controllers)</parameters>
-					<controller_manager_node_name>controller_manager</controller_manager_node_name>
-			</plugin>
-			<plugin filename="libignition-gazebo-sensors-system.so" name="ignition::gazebo::systems::Sensors">
-					<render_engine>$(arg gazebo_renderer)</render_engine>
-			</plugin>
-		</gazebo>
-		<gazebo reference="camera_color_frame">
-			<sensor name="camera_sensor" type="rgbd_camera">
-				<camera>
-					<horizontal_fov>1.047</horizontal_fov>
-					<image>
-						<width>$(arg camera_width)</width>
-						<height>$(arg camera_height)</height>
-						<format>RGB_INT8</format>
-					</image>
-					<clip>
-						<near>0.1</near>
-						<far>5</far>
-					</clip>
-					<distortion>
-						<k1>0.0</k1>
-						<k2>0.0</k2>
-						<k3>0.0</k3>
-						<p1>0.0</p1>
-						<p2>0.0</p2>
-						<center>0.5 0.5</center>
-					</distortion>
-					<lens>
-						<intrinsics>
-							<fx>554.25469</fx>
-							<fy>554.25469</fy>
-							<cx>320.5</cx>
-							<cy>240.5</cy>
-							<s>0</s>
-						</intrinsics>
-						<!-- These need to match the intrinsics above or
-						Ignition will default to different default values -->
-						<projection>
-							<p_fx>554.25469</p_fx>
-							<p_fy>554.25469</p_fy>
-							<p_cx>320.5</p_cx>
-							<p_cy>240.5</p_cy>
-							<tx>0</tx>
-							<ty>0</ty>
-						</projection>
-					</lens>
-					<noise>
-						<type>gaussian</type>
-						<mean>0</mean>
-						<stddev>0.00</stddev>
-					</noise>
-					<depth_camera>
-						<clip>
-						<near>0.25</near>
-						<far>5</far>
-						</clip>
-					</depth_camera>
-					<optical_frame_id>color_optical_frame</optical_frame_id>
-				</camera>
-				<ignition_frame_id>camera_color_frame</ignition_frame_id>
-				<always_on>1</always_on>
-				<update_rate>$(arg camera_fps)</update_rate>
-				<visualize>true</visualize>
-				<topic>wrist_mounted_camera</topic>
-				<enable_metrics>false</enable_metrics>
-			</sensor>
-		</gazebo>
-	</xacro:if>
 </robot>
