Commit message: 1030

File: mobile_manipulator/urdf/camera.xacro (robot description, xacro)
@@ -21,5 +21,4 @@
   <xacro:property name="rgb_horizontal_fov" value="${69.4 * M_PI / 180}"/>
   <xacro:property name="depth_horizontal_fov" value="${85.2 * M_PI / 180}"/>
-  <xacro:include filename="$(find mobile_manipulator)/urdf/gazebo_settings.xacro"/>
   <xacro:macro name="camera" params="
     parent
@@ -78,12 +77,63 @@
       </joint>
       <link name="${parent}_color_optical_frame"/>
-      <xacro:gazebo_camera
-        camera_frame="${parent}"
-        color_camera_optical_frame="${parent}_color_optical_frame"
-        depth_camera_optical_frame="${parent}_depth_optical_frame"
-        camera_width="${camera_width}"
-        camera_height="${camera_height}"
-        camera_fps="${camera_fps}"
-        horizontal_fov="${rgb_horizontal_fov}"/>
+      <joint name="${parent}_infra1_joint" type="fixed">
+        <origin xyz="0 ${d435_cam_depth_to_infra1_offset} 0" rpy="0 0 0" />
+        <parent link="${parent}_depth_frame" />
+        <child link="${parent}_infra1_frame" />
+      </joint>
+      <link name="${parent}_infra1_frame"/>
+      <joint name="${parent}_infra1_optical_joint" type="fixed">
+        <origin xyz="0 0 0" rpy="${-M_PI/2} 0 ${-M_PI/2}" />
+        <parent link="${parent}_infra1_frame" />
+        <child link="${parent}_infra1_optical_frame" />
+      </joint>
+      <link name="${parent}_infra1_optical_frame"/>
+      <joint name="${parent}_infra2_joint" type="fixed">
+        <origin xyz="0 ${d435_cam_depth_to_infra2_offset} 0" rpy="0 0 0" />
+        <parent link="${parent}_depth_frame" />
+        <child link="${parent}_infra2_frame" />
+      </joint>
+      <link name="${parent}_infra2_frame"/>
+      <joint name="${parent}_infra2_optical_joint" type="fixed">
+        <origin xyz="0 0 0" rpy="${-M_PI/2} 0 ${-M_PI/2}" />
+        <parent link="${parent}_infra2_frame" />
+        <child link="${parent}_infra2_optical_frame" />
+      </joint>
+      <link name="${parent}_infra2_optical_frame"/>
+      <joint name="${parent}_accel_joint" type="fixed">
+        <origin xyz = "-0.01174 -0.00552 0.0051" rpy = "0 0 0" />
+        <parent link="${parent}_depth_frame" />
+        <child link="${parent}_accel_frame" />
+      </joint>
+      <link name="${parent}_accel_frame"/>
+      <joint name="${parent}_accel_optical_joint" type="fixed">
+        <origin xyz = "0 0 0" rpy = "${-M_PI/2} 0 ${-M_PI/2}" />
+        <parent link="${parent}_accel_frame" />
+        <child link="${parent}_accel_optical_frame" />
+      </joint>
+      <link name="${parent}_accel_optical_frame"/>
+      <joint name="${parent}_gyro_joint" type="fixed">
+        <origin xyz = "-0.01174 -0.00552 0.0051" rpy = "0 0 0" />
+        <parent link="${parent}_depth_frame" />
+        <child link="${parent}_gyro_frame" />
+      </joint>
+      <link name="${parent}_gyro_frame"/>
+      <joint name="${parent}_gyro_optical_joint" type="fixed">
+        <origin xyz = "0 0 0" rpy = "${-M_PI/2} 0 ${-M_PI/2}" />
+        <parent link="${parent}_gyro_frame" />
+        <child link="${parent}_gyro_optical_frame" />
+      </joint>
+      <link name="${parent}_gyro_optical_frame"/>
+      <xacro:if value="${sim_gazebo}">
+        <xacro:include filename="$(find mobile_manipulator)/urdf/gazebo_camera.xacro"/>
+        <xacro:gazebo_camera
+          camera_frame="${parent}"
+          color_camera_optical_frame="${parent}_color_optical_frame"
+          depth_camera_optical_frame="${parent}_depth_optical_frame"
+          camera_width="${camera_width}"
+          camera_height="${camera_height}"
+          camera_fps="${camera_fps}"
+          horizontal_fov="${rgb_horizontal_fov}"/>
+      </xacro:if>
     </xacro:if>
   </xacro:macro>

File: mobile_manipulator/urdf/gazebo_settings.xacro (robot description, xacro)
@@ -1,96 +1,114 @@
 <?xml version="1.0"?>
 <robot xmlns:xacro="http://www.ros.org/wiki/xacro">
-  <xacro:property name="M_PI" value="3.14159265358979323846" />
-	<xacro:macro name="gazebo_lidar" params="
-		parent">
-		<gazebo reference="${parent}">
-			<material>Gazebo/Black</material>
-			<sensor name="2d_lidar" type="gpu_ray">
-				<pose>0 0 0 0 0 0</pose>
-				<visualize>true</visualize>
-				<update_rate>10</update_rate>
-				<ray>
-					<scan>
-						<horizontal>
-							<samples>720</samples>
-							<resolution>1</resolution>
-							<min_angle>-${M_PI}</min_angle>
-							<max_angle>${M_PI}</max_angle>
-						</horizontal>
-					</scan>
-					<range>
-						<min>0.1</min>
-						<max>12.0</max>
-						<resolution>0.01</resolution>
-					</range>
-				</ray>
-				<plugin name="gazebo_ros_lidar" filename="libgazebo_ros_ray_sensor.so">
-					<output_type>sensor_msgs/LaserScan</output_type>
-					<frame_name>${parent}</frame_name>
-				</plugin>
-			</sensor>
-		</gazebo>
-	</xacro:macro>
-	<xacro:macro name="gazebo_camera" params="
-		camera_frame
-		color_camera_optical_frame
-		depth_camera_optical_frame
-		camera_width
-		camera_height
-		camera_fps
-		horizontal_fov">
-		<gazebo reference="${camera_frame}_color_frame">
-			<sensor name="${camera_frame}_color_sensor" type="camera">
-				<pose>0 0 0 0 0 0</pose>
-				<always_on>1</always_on>
-				<visualize>true</visualize>
-				<update_rate>${camera_fps}</update_rate>
-				<camera>
-					<horizontal_fov>${horizontal_fov}</horizontal_fov>
-					<image>
-						<format>R8G8B8</format>
-						<width>${camera_width}</width>
-						<height>${camera_height}</height>
-					</image>
-					<clip>
-						<near>0.05</near>
-						<far>10.0</far>
-					</clip>
-				</camera>
-				<plugin name="${camera_frame}_color_controller" filename="libgazebo_ros_camera.so">
-					<frame_name>${color_camera_optical_frame}</frame_name>
-					<image_topic>${camera_frame}/color/image_raw</image_topic>
-					<camera_info_topic>${camera_frame}/color/camera_info</camera_info_topic>
-				</plugin>
-			</sensor>
-		</gazebo>
-		<gazebo reference="${camera_frame}_depth_frame">
-			<sensor name="${camera_frame}_depth_sensor" type="depth">
-				<pose>0 0 0 0 0 0</pose>
-				<always_on>1</always_on>
-				<visualize>true</visualize>
-				<update_rate>${camera_fps}</update_rate>
-				<camera>
-					<horizontal_fov>${horizontal_fov}</horizontal_fov>
-					<image>
-						<format>B8G8R8</format>
-						<width>${camera_width}</width>
-						<height>${camera_height}</height>
-					</image>
-					<clip>
-						<near>0.05</near>
-						<far>10.0</far>
-					</clip>
-				</camera>
-				<plugin name="${camera_frame}_depth" filename="libgazebo_ros_camera.so">
-					<frame_name>${depth_camera_optical_frame}</frame_name>
-					<min_depth>0.1</min_depth>
-					<max_depth>10.0</max_depth>
-					<image_topic>${camera_frame}/depth/image_raw</image_topic>
-					<camera_info_topic>${camera_frame}/depth/camera_info</camera_info_topic>
-					<point_cloud_topic>${camera_frame}/depth/points</point_cloud_topic>
-				</plugin>
-			</sensor>
-		</gazebo>
-	</xacro:macro>
+  <xacro:macro name="gazebo_kinematics" params="
+    reference
+    r g b
+    mu1
+    mu2
+    restitution_coefficient
+    kp
+    kd
+    max_vel
+    min_depth">
+    <gazebo reference="${reference}">
+      <visual>
+        <material>
+          <diffuse>${r} ${g} ${b} 1.0</diffuse>
+          <ambient>${r} ${g} ${b} 1.0</ambient>
+          <specular>${r} ${g} ${b} 1.0</specular>
+        </material>
+      </visual>
+      <surface>
+        <friction>
+          <ode>
+            <mu1>${mu1}</mu1>
+            <mu2>${mu2}</mu2>
+          </ode>
+        </friction>
+        <bounce>
+          <restitution_coefficient>${restitution_coefficient}</restitution_coefficient>
+        </bounce>
+        <contact>
+          <ode>
+            <kp>${kp}</kp>
+            <kd>${kd}</kd>
+            <max_vel>${max_vel}</max_vel>
+            <min_depth>${min_depth}</min_depth>
+          </ode>
+        </contact>
+      </surface>
+    </gazebo>
+  </xacro:macro>
+	<gazebo reference="base_body">
+    <visual>
+      <material>
+        <diffuse>0.9 0.9 0.9 1</diffuse>
+        <ambient>0.9 0.9 0.9 1</ambient>
+        <specular>0.9 0.9 0.9 1</specular>
+      </material>
+    </visual>
+  </gazebo>
+  <gazebo reference="camera_case_link">
+    <visual>
+      <material>
+        <diffuse>0.1 0.1 0.1 1</diffuse>
+        <ambient>0.1 0.1 0.1 1</ambient>
+        <specular>0.1 0.1 0.1 1</specular>
+      </material>
+    </visual>
+  </gazebo>
+  <xacro:gazebo_kinematics reference="fr_wheel"
+    r="0.175" g="0.175" b="0.175"
+    mu1="200"
+    mu2="200"
+    restitution_coefficient="0.0"
+    kp="100000.0"
+    kd="100.0"
+    max_vel="0.01"
+    min_depth="0.001"/>
+  <xacro:gazebo_kinematics reference="fl_wheel"
+    r="0.175" g="0.175" b="0.175"
+    mu1="200"
+    mu2="200"
+    restitution_coefficient="0.0"
+    kp="100000.0"
+    kd="100.0"
+    max_vel="0.01"
+    min_depth="0.001"/>
+  <xacro:gazebo_kinematics reference="rl_bracket"
+    r="0.175" g="0.175" b="0.175"
+    mu1="100"
+    mu2="100"
+    restitution_coefficient="0.0"
+    kp="100000.0"
+    kd="100.0"
+    max_vel="0.01"
+    min_depth="0.001"/>
+  <xacro:gazebo_kinematics reference="rl_wheel"
+    r="0.175" g="0.175" b="0.175"
+    mu1="200"
+    mu2="200"
+    restitution_coefficient="0.0"
+    kp="100000.0"
+    kd="100.0"
+    max_vel="0.01"
+    min_depth="0.001"/>
+  <xacro:gazebo_kinematics reference="rr_bracket"
+    r="0.175" g="0.175" b="0.175"
+    mu1="100"
+    mu2="100"
+    restitution_coefficient="0.0"
+    kp="100000.0"
+    kd="100.0"
+    max_vel="0.01"
+    min_depth="0.001"/>
+  <xacro:gazebo_kinematics reference="rr_wheel"
+    r="0.175" g="0.175" b="0.175"
+    mu1="200"
+    mu2="200"
+    restitution_coefficient="0.0"
+    kp="100000.0"
+    kd="100.0"
+    max_vel="0.01"
+    min_depth="0.001"/>
 </robot>

File: mobile_manipulator/urdf/integrate_execution.xacro (robot description, xacro)
@@ -12,6 +12,6 @@
 	<xacro:arg name="use_fake_hardware" default="false"/>
 	<xacro:arg name="fake_sensor_commands" default="false"/>
-	<xacro:arg name="sim_gazebo" default="true"/>
-	<xacro:arg name="sim_ignition" default="false"/>
+	<xacro:arg name="sim_gazebo" default="false"/>
+	<xacro:arg name="sim_ignition" default="true"/>
 	<xacro:arg name="sim_isaac" default="false"/>
 	<xacro:arg name="gripper_joint_name" default="right_finger_bottom_joint"/>
@@ -24,11 +24,13 @@
 	<xacro:arg name="simulation_controllers" default="$(find mobile_manipulator)/config/ros2_control.yaml"/>
 	<xacro:arg name="initial_value" default="$(find mobile_manipulator)/config/initial_value.yaml"/>
+	<xacro:arg name="select_camera" default="both"/>
 	<xacro:property name="initial_value" default="$(arg initial_value)"/>
-  <xacro:property name="camera_width" value="1280"/>
-  <xacro:property name="camera_height" value="720"/>
-  <xacro:property name="camera_fps" value="30"/>
-  <xacro:property name="M_PI" value="3.1415926535897931" />
-  <xacro:property name="horizontal_fov" value="${69.4 * M_PI / 180}"/>
 	<xacro:include filename="$(find mobile_manipulator)/urdf/integrate_model.xacro"/>
+	<xacro:if value="$(arg sim_ignition)">
+		<xacro:property name="root_link" default="world"/>
+	</xacro:if>
+	<xacro:unless value="$(arg sim_ignition)">
+		<xacro:property name="root_link" default="base_link"/>
+	</xacro:unless>
 	<xacro:load_model
 		vision="$(arg vision)"
@@ -51,5 +53,7 @@
 		isaac_joint_commands="$(arg isaac_joint_commands)"
 		isaac_joint_states="$(arg isaac_joint_states)"
-		initial_value="${xacro.load_yaml(initial_value)}"/>
+		initial_value="${xacro.load_yaml(initial_value)}"
+		select_camera="$(arg select_camera)"
+		root_link="${root_link}"/>
 	<xacro:if value="$(arg sim_gazebo)">
 		<gazebo>
@@ -63,5 +67,5 @@
 			<plugin filename="libign_ros2_control-system.so" name="ign_ros2_control::IgnitionROS2ControlPlugin">
 				<namespace>/</namespace>
-				<parameters>$(arg simulation_controllers)</parameters>
+				<parameters>$(find mobile_manipulator)/config/ros2_control.yaml</parameters>
 				<controller_manager_node_name>controller_manager</controller_manager_node_name>
 			</plugin>
@@ -69,5 +73,6 @@
 				<render_engine>$(arg gazebo_renderer)</render_engine>
 			</plugin>
-		</gazebo>
+    	<plugin filename="ignition-gazebo-joint-state-publisher-system" name="ignition::gazebo::systems::JointStatePublisher"/>
+  	</gazebo>
 	</xacro:if>
 </robot>
