Commit message: 1010

File: mobile_manipulator/urdf/integrate_model.xacro (robot description, xacro)
@@ -12,10 +12,10 @@
   <xacro:property name="rear_wheel_depth" value="0.022335230282742743" />
   <xacro:property name="base_body_mass" value="24.3948952632956" />
-  <xacro:property name="front_wheel_mass" value="1.0568406891164" />
-  <xacro:property name="rear_wheel_bracket_mass" value="0.0211573699864" />
-  <xacro:property name="rear_wheel_mass" value="0.0920111896829" />
-  <xacro:property name="camera_mass" value="0.2333248928640" />
-  <xacro:property name="lidar_mass" value="0.1071556446529" />
-  <xacro:property name="base_arm_connector_mass" value="0.4535071053510" />
+  <xacro:property name="front_wheel_mass" value="1.0" />
+  <xacro:property name="rear_wheel_bracket_mass" value="0.2" />
+  <xacro:property name="rear_wheel_mass" value="0.1" />
+  <xacro:property name="base_arm_connector_mass" value="0.3" />
+  <xacro:property name="camera_mass" value="0.072" />
+  <xacro:property name="lidar_mass" value="0.1" />
   <!-- Include inertial xacro files -->
   <xacro:include filename="$(find mobile_manipulator)/urdf/inertial.xacro" />
@@ -41,15 +41,15 @@
     isaac_joint_states
     initial_value">
-    <!-- Ros2 Control Include -->
+    <xacro:include filename="$(find mobile_manipulator)/urdf/camera.xacro"/>
     <xacro:include filename="$(find mobile_manipulator)/urdf/integrate_ros2_control.xacro" />
-      <xacro:mobile_manipulator_control
-        use_fake_hardware="${use_fake_hardware}"
-        fake_sensor_commands="${fake_sensor_commands}"
-        sim_gazebo="${sim_gazebo}"
-        sim_ignition="${sim_ignition}"
-        sim_isaac="${sim_isaac}"
-        isaac_joint_commands="${isaac_joint_commands}"
-        isaac_joint_states="${isaac_joint_states}"
-        initial_value="${initial_value}"/>
+    <xacro:mobile_manipulator_control
+      use_fake_hardware="${use_fake_hardware}"
+      fake_sensor_commands="${fake_sensor_commands}"
+      sim_gazebo="${sim_gazebo}"
+      sim_ignition="${sim_ignition}"
+      sim_isaac="${sim_isaac}"
+      isaac_joint_commands="${isaac_joint_commands}"
+      isaac_joint_states="${isaac_joint_states}"
+      initial_value="${initial_value}"/>
     <link name="base_link"/>
     <joint name="base_body_joint" type="fixed">
@@ -57,5 +57,4 @@
       <parent link="base_link" />
       <child link="base_body" />
-      <axis xyz="0 0 0" />
     </joint>
     <link name="base_body">
@@ -63,5 +62,5 @@
         <origin xyz="0 0 0" rpy="0 0 0" />
         <geometry>
-          <mesh filename="package://mobile_manipulator/meshes/base/base_body.stl" />
+          <mesh filename="$(find mobile_manipulator)/meshes/base/base_body.stl" />
         </geometry>
         <material name="">
@@ -72,5 +71,5 @@
         <origin xyz="0 0 0" rpy="0 0 0" />
         <geometry>
-          <mesh filename="package://mobile_manipulator/meshes/base/base_body.stl" />
+          <mesh filename="$(find mobile_manipulator)/meshes/base/base_body.stl" />
         </geometry>
       </collision>
@@ -89,5 +88,5 @@
         <origin rpy="${M_PI/2} 0 0" xyz="0 0 0" />
         <geometry>
-          <mesh filename="package://mobile_manipulator/meshes/base/front_wheel.stl" />
+          <mesh filename="$(find mobile_manipulator)/meshes/base/front_wheel.stl" />
         </geometry>
         <material name="">
@@ -98,5 +97,5 @@
         <origin rpy="${M_PI/2} 0 0" xyz="0 0 0" />
         <geometry>
-          <mesh filename="package://mobile_manipulator/meshes/base/front_wheel.stl" />
+          <mesh filename="$(find mobile_manipulator)/meshes/base/front_wheel.stl" />
         </geometry>
       </collision>
@@ -115,5 +114,5 @@
         <origin rpy="-${M_PI/2} 0 0" xyz="0 0 0" />
         <geometry>
-          <mesh filename="package://mobile_manipulator/meshes/base/front_wheel.stl" />
+          <mesh filename="$(find mobile_manipulator)/meshes/base/front_wheel.stl" />
         </geometry>
         <material name="">
@@ -124,5 +123,5 @@
         <origin rpy="-${M_PI/2} 0 0" xyz="0 0 0" />
         <geometry>
-          <mesh filename="package://mobile_manipulator/meshes/base/front_wheel.stl" />
+          <mesh filename="$(find mobile_manipulator)/meshes/base/front_wheel.stl" />
         </geometry>
       </collision>
@@ -141,5 +140,5 @@
         <origin rpy="0 0 ${M_PI/2}" xyz="0 0 0" />
         <geometry>
-          <mesh filename="package://mobile_manipulator/meshes/base/rear_wheel_bracket.stl" />
+          <mesh filename="$(find mobile_manipulator)/meshes/base/rear_wheel_bracket.stl" />
         </geometry>
         <material name="">
@@ -150,5 +149,5 @@
         <origin rpy="0 0 ${M_PI/2}" xyz="0 0 0" />
         <geometry>
-          <mesh filename="package://mobile_manipulator/meshes/base/rear_wheel_bracket.stl" />
+          <mesh filename="$(find mobile_manipulator)/meshes/base/rear_wheel_bracket.stl" />
         </geometry>
       </collision>
@@ -167,5 +166,5 @@
         <origin rpy="0 -${M_PI/2} 0" xyz="0 0 0" />
         <geometry>
-          <mesh filename="package://mobile_manipulator/meshes/base/rear_wheel.stl" />
+          <mesh filename="$(find mobile_manipulator)/meshes/base/rear_wheel.stl" />
         </geometry>
         <material name="">
@@ -176,5 +175,5 @@
         <origin rpy="0 -${M_PI/2} 0" xyz="0 0 0" />
         <geometry>
-          <mesh filename="package://mobile_manipulator/meshes/base/rear_wheel.stl" />
+          <mesh filename="$(find mobile_manipulator)/meshes/base/rear_wheel.stl" />
         </geometry>
       </collision>
@@ -193,5 +192,5 @@
         <origin rpy="0 0 ${M_PI/2}" xyz="0 0 0" />
         <geometry>
-          <mesh filename="package://mobile_manipulator/meshes/base/rear_wheel_bracket.stl" />
+          <mesh filename="$(find mobile_manipulator)/meshes/base/rear_wheel_bracket.stl" />
         </geometry>
         <material name="">
@@ -202,5 +201,5 @@
         <origin rpy="0 0 ${M_PI/2}" xyz="0 0 0" />
         <geometry>
-          <mesh filename="package://mobile_manipulator/meshes/base/rear_wheel_bracket.stl" />
+          <mesh filename="$(find mobile_manipulator)/meshes/base/rear_wheel_bracket.stl" />
         </geometry>
       </collision>
@@ -219,5 +218,5 @@
         <origin rpy="0 ${M_PI/2} 0" xyz="0 0 0" />
         <geometry>
-          <mesh filename="package://mobile_manipulator/meshes/base/rear_wheel.stl" />
+          <mesh filename="$(find mobile_manipulator)/meshes/base/rear_wheel.stl" />
         </geometry>
         <material name="">
@@ -228,5 +227,5 @@
         <origin rpy="0 ${M_PI/2} 0" xyz="0 0 0" />
         <geometry>
-          <mesh filename="package://mobile_manipulator/meshes/base/rear_wheel.stl" />
+          <mesh filename="$(find mobile_manipulator)/meshes/base/rear_wheel.stl" />
         </geometry>
       </collision>
@@ -239,5 +238,4 @@
       <parent link="base_body" />
       <child link="laser_Link" />
-      <axis xyz="0 0 0" />
     </joint>
     <link name="laser_Link">
@@ -245,5 +243,5 @@
         <origin xyz="0 0 0" rpy="0 0 0" />
         <geometry>
-          <mesh filename="package://mobile_manipulator/meshes/base/lidar.stl" />
+          <mesh filename="$(find mobile_manipulator)/meshes/base/lidar.stl" />
         </geometry>
         <material name="">
@@ -254,5 +252,5 @@
         <origin xyz="0 0 0" rpy="0 0 0" />
         <geometry>
-          <mesh filename="package://mobile_manipulator/meshes/base/lidar.stl" />
+          <mesh filename="$(find mobile_manipulator)/meshes/base/lidar.stl" />
         </geometry>
       </collision>
@@ -264,32 +262,35 @@
       <origin xyz="0.115 0 -0.04565" rpy="0 0 0" />
       <parent link="base_body" />
-      <child link="base_camera_link" />
-      <axis xyz="0 0 0" />
-    </joint>
-    <link name="base_camera_link">
-      <visual>
-        <origin xyz="0 0 0" rpy="0 0 0" />
-        <geometry>
-          <mesh filename="package://mobile_manipulator/meshes/base/camera.stl" />
-        </geometry>
-        <material name="">
-          <color rgba="0.79216 0.81961 0.93333 1" />
-        </material>
-      </visual>
-      <collision>
-        <origin xyz="0 0 0" rpy="0 0 0" />
-        <geometry>
-          <mesh filename="package://mobile_manipulator/meshes/base/camera.stl" />
-        </geometry>
-      </collision>
-      <xacro:inertial_cylinder mass="${camera_mass}" length="0.08832" radius="0.01265">
-        <origin xyz="0 0 0" rpy="-${M_PI/2} 0 0" />
-      </xacro:inertial_cylinder>
-    </link>
+      <child link="base_camera" />
+    </joint>
+    <link name="base_camera">
+      <visual>
+        <origin xyz="0 0 0" rpy="${M_PI/2} 0 ${M_PI/2}" />
+        <geometry>
+          <mesh filename="$(find mobile_manipulator)/meshes/base/d435.dae" />
+        </geometry>
+        <material name="aluminum">
+          <color rgba="0.5 0.5 0.5 1" />
+        </material>
+      </visual>
+      <collision>
+        <origin xyz="0 0 0" rpy="${M_PI/2} 0 ${M_PI/2}" />
+        <geometry>
+          <mesh filename="$(find mobile_manipulator)/meshes/base/d435.dae" />
+        </geometry>
+      </collision>
+      <xacro:inertial_box mass="${camera_mass}" x="0.090" y="0.02505" z="0.025">
+        <origin xyz="0 0 0" rpy="${M_PI/2} 0 ${M_PI/2}" />
+      </xacro:inertial_box>
+    </link>
+    <xacro:camera
+      parent="base_camera"
+      sim_gazebo="${sim_gazebo}"
+      sim_ignition="${sim_ignition}"
+      sim_isaac="${sim_isaac}"/>
     <joint name="base_arm_connector_joint" type="fixed">
       <origin xyz="0 0 0.0576" rpy="0 0 0" />
       <parent link="base_body" />
       <child link="base_arm_connector"/>
-      <axis xyz="0 0 0" />
     </joint>
     <link name="base_arm_connector">
@@ -297,5 +298,5 @@
         <origin xyz="0 0 -0.0288" rpy="0 0 0" />
         <geometry>
-          <mesh filename="package://mobile_manipulator/meshes/base/base_arm_connector.stl" />
+          <mesh filename="$(find mobile_manipulator)/meshes/base/base_arm_connector.stl" />
         </geometry>
         <material name="">
@@ -306,5 +307,5 @@
         <origin xyz="0 0 -0.0288" rpy="0 0 0" />
         <geometry>
-          <mesh filename="package://mobile_manipulator/meshes/base/base_arm_connector.stl" />
+          <mesh filename="$(find mobile_manipulator)/meshes/base/base_arm_connector.stl" />
         </geometry>
       </collision>
@@ -325,5 +326,5 @@
         <origin xyz="0 0 0" rpy="0 0 0" />
         <geometry>
-          <mesh filename="package://mobile_manipulator/meshes/arm/base_link.STL" />
+          <mesh filename="$(find mobile_manipulator)/meshes/arm/base_link.STL" />
         </geometry>
         <material name="">
@@ -334,5 +335,5 @@
         <origin xyz="0 0 0" rpy="0 0 0" />
         <geometry>
-          <mesh filename="package://mobile_manipulator/meshes/arm/base_link.STL" />
+          <mesh filename="$(find mobile_manipulator)/meshes/arm/base_link.STL" />
         </geometry>
       </collision>
@@ -357,5 +358,5 @@
         <origin xyz="0 0 0" rpy="0 0 0" />
         <geometry>
-          <mesh filename="package://mobile_manipulator/meshes/arm/shoulder_link.STL" />
+          <mesh filename="$(find mobile_manipulator)/meshes/arm/shoulder_link.STL" />
         </geometry>
         <material name="">
@@ -366,5 +367,5 @@
         <origin xyz="0 0 0" rpy="0 0 0" />
         <geometry>
-          <mesh filename="package://mobile_manipulator/meshes/arm/shoulder_link.STL" />
+          <mesh filename="$(find mobile_manipulator)/meshes/arm/shoulder_link.STL" />
         </geometry>
       </collision>
@@ -379,5 +380,5 @@
     </gazebo>
 		<joint name="arm_joint_2" type="revolute">
-      <origin xyz="0 -0.03 0.115" rpy="1.5708 0 0" />
+      <origin xyz="0 -0.03 0.115" rpy="${M_PI/2} 0 0" />
       <parent link="arm_link_1" />
       <child link="arm_link_2" />
@@ -386,4 +387,19 @@
     </joint>
     <link name="arm_link_2">
+      <visual>
+        <origin xyz="0 0 0" rpy="0 0 0" />
+        <geometry>
+          <mesh filename="$(find mobile_manipulator)/meshes/arm/arm_link.STL" />
+        </geometry>
+        <material name="">
+          <color rgba="0.803 0.824 0.820 1" />
+        </material>
+      </visual>
+      <collision>
+        <origin xyz="0 0 0" rpy="0 0 0" />
+        <geometry>
+          <mesh filename="$(find mobile_manipulator)/meshes/arm/arm_link.STL" />
+        </geometry>
+      </collision>
       <inertial>
         <origin xyz="0.02998299 0.21154808 0.0453031" rpy="0 0 0" />
@@ -391,19 +407,4 @@
         <inertia ixx="0.01149277" ixy="1E-06" ixz="1.6E-07" iyy="0.00102851" iyz="0.00140765" izz="0.01133492" />
       </inertial>
-      <visual>
-        <origin xyz="0 0 0" rpy="0 0 0" />
-        <geometry>
-          <mesh filename="package://mobile_manipulator/meshes/arm/arm_link.STL" />
-        </geometry>
-        <material name="">
-          <color rgba="0.803 0.824 0.820 1" />
-        </material>
-      </visual>
-      <collision>
-        <origin xyz="0 0 0" rpy="0 0 0" />
-        <geometry>
-          <mesh filename="package://mobile_manipulator/meshes/arm/arm_link.STL" />
-        </geometry>
-      </collision>
     </link>
     <gazebo reference="arm_link_2">
@@ -411,5 +412,5 @@
     </gazebo>
     <joint name="arm_joint_3" type="revolute">
-      <origin xyz="0 0.28 0" rpy="-3.1416 0 0" />
+      <origin xyz="0 0.28 0" rpy="-${M_PI} 0 0" />
       <parent link="arm_link_2" />
       <child link="arm_link_3" />
@@ -418,4 +419,19 @@
     </joint>
     <link name="arm_link_3">
+      <visual>
+        <origin xyz="0 0 0" rpy="0 0 0" />
+        <geometry>
+          <mesh filename="$(find mobile_manipulator)/meshes/arm/forearm_link.STL" />
+        </geometry>
+        <material name="">
+          <color rgba="0.803 0.824 0.820 1" />
+        </material>
+      </visual>
+      <collision>
+        <origin xyz="0 0 0" rpy="0 0 0" />
+        <geometry>
+          <mesh filename="$(find mobile_manipulator)/meshes/arm/forearm_link.STL" />
+        </geometry>
+      </collision>
       <inertial>
         <origin xyz="0.0301559 0.09502206 0.0073555" rpy="0 0 0" />
@@ -423,19 +439,4 @@
         <inertia ixx="0.00163256" ixy="7.11E-06" ixz="1.54E-06" iyy="0.00029798" iyz="9.587E-05" izz="0.00169091" />
       </inertial>
-      <visual>
-        <origin xyz="0 0 0" rpy="0 0 0" />
-        <geometry>
-          <mesh filename="package://mobile_manipulator/meshes/arm/forearm_link.STL" />
-        </geometry>
-        <material name="">
-          <color rgba="0.803 0.824 0.820 1" />
-        </material>
-      </visual>
-      <collision>
-        <origin xyz="0 0 0" rpy="0 0 0" />
-        <geometry>
-          <mesh filename="package://mobile_manipulator/meshes/arm/forearm_link.STL" />
-        </geometry>
-      </collision>
     </link>
     <gazebo reference="arm_link_3">
@@ -443,5 +444,5 @@
     </gazebo>
 		<joint name="arm_joint_4" type="revolute">
-      <origin xyz="0 -0.14 0.02" rpy="1.5708 0 0" />
+      <origin xyz="0 -0.14 0.02" rpy="${M_PI/2} 0 0" />
       <parent link="arm_link_3" />
       <child link="arm_link_4" />
@@ -450,4 +451,19 @@
     </joint>
     <link name="arm_link_4">
+      <visual>
+        <origin xyz="0 0 0" rpy="0 0 0" />
+        <geometry>
+          <mesh filename="$(find mobile_manipulator)/meshes/arm/lower_wrist_link.STL" />
+        </geometry>
+        <material name="">
+          <color rgba="0.803 0.824 0.820 1" />
+        </material>
+      </visual>
+      <collision>
+        <origin xyz="0 0 0" rpy="0 0 0" />
+        <geometry>
+          <mesh filename="$(find mobile_manipulator)/meshes/arm/lower_wrist_link.STL" />
+        </geometry>
+      </collision>
       <inertial>
         <origin xyz="0.00575149 0.01000443 0.08719207" rpy="0 0 0" />
@@ -455,19 +471,4 @@
         <inertia ixx="0.00069098" ixy="2.4E-07" ixz="0.00016483" iyy="0.00078519" iyz="7.4E-07" izz="0.00034115" />
       </inertial>
-      <visual>
-        <origin xyz="0 0 0" rpy="0 0 0" />
-        <geometry>
-          <mesh filename="package://mobile_manipulator/meshes/arm/lower_wrist_link.STL" />
-        </geometry>
-        <material name="">
-          <color rgba="0.803 0.824 0.820 1" />
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
Commit message: 1102

File: mobile_manipulator/urdf/integrate_model.xacro (robot description, xacro)
@@ -85,5 +85,5 @@
         <origin xyz="0 0 0" rpy="0 0 0" />
         <geometry>
-          <mesh filename="file://$(find mobile_manipulator)/meshes/base/base_body.dae" />
+          <mesh filename="file://$(find mobile_manipulator)/meshes/base/base_body.stl" />
         </geometry>
         <material name="">
@@ -94,5 +94,5 @@
         <origin xyz="0 0 0" rpy="0 0 0" />
         <geometry>
-          <mesh filename="file://$(find mobile_manipulator)/meshes/base/base_body.dae" />
+          <mesh filename="file://$(find mobile_manipulator)/meshes/base/base_body.stl" />
         </geometry>
       </collision>
